File: TakpadV6.1.brd (EAGLE design)
At the start: 102.6 x 100.1 mm, 68 parts, among them J1 SD_CARD_SOCKET, J10 AUDIO_JACK_TRRSSMD_RA, J3 AVR_SPI_PROG_3X2PTH, T1 0, T2 0, T3 0, U1 ATMEGA328P_TQFP, U4 LM386N, Y1 20MHz

Commit message: Add files via upload
Minor Changes
Parts:
- moved C13 1.87 mm to (1.90, 13.0)
- moved J2 1.70 mm to (1.96, 6.40)
Connections:
- net V+: now also U1.18
Routing:
- net V+: track 126.1 -> 128.5 mm
- net VIN: track 39.3 -> 41.0 mm
- net N$7: track 10.1 -> 9.60 mm
Changed lines of the file:
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@@
 <?xml version="1.0" encoding="utf-8"?>
 <!DOCTYPE eagle SYSTEM "eagle.dtd">
-<eagle version="8.4.1">
+<eagle version="8.4.0">
 <drawing>
 <settings>
@@
 <param name="dpMaxLengthDifference" value="10mm"/>
 <param name="dpGapFactor" value="2.5"/>
-<param name="checkAngle" value="0"/>
 <param name="checkFont" value="1"/>
 <param name="checkRestrict" value="1"/>
@@
 <attribute name="VALUE" x="18.36" y="2.0475" size="0.6096" layer="27" font="vector" ratio="20" align="top-center"/>
 </element>
-<element name="J2" library="SparkFun-Connectors" library_urn="urn:adsk.eagle:library:513" package="USB-B-MICRO-SMD_RED_PASTE" package3d_urn="urn:adsk.eagle:package:38239/1" value="" x="3.66" y="6.4" smashed="yes">
-<attribute name="NAME" x="2.39" y="11.2006" size="1.27" layer="25" font="vector" ratio="20"/>
-<attribute name="PROD_ID" value="CONN-11752" x="3.66" y="6.4" size="1.778" layer="27" display="off"/>
-<attribute name="VALUE" x="2.39" y="1.5994" size="0.6096" layer="27" font="vector" ratio="20" align="top-left"/>
+<element name="J2" library="SparkFun-Connectors" library_urn="urn:adsk.eagle:library:513" package="USB-B-MICRO-SMD_RED_PASTE" package3d_urn="urn:adsk.eagle:package:38239/1" value="" x="1.96" y="6.4" smashed="yes">
+<attribute name="NAME" x="0.69" y="11.2006" size="1.27" layer="25" font="vector" ratio="20"/>
+<attribute name="PROD_ID" value="CONN-11752" x="1.96" y="6.4" size="1.778" layer="27" display="off"/>
+<attribute name="VALUE" x="0.69" y="1.5994" size="0.6096" layer="27" font="vector" ratio="20" align="top-left"/>
 </element>
 <element name="D7" library="SparkFun-LED" library_urn="urn:adsk.eagle:library:529" package="LED-1206" package3d_urn="urn:adsk.eagle:package:39352/1" value="GREEN" x="18.36" y="7.7" smashed="yes">
@@
 <attribute name="VALUE" x="25.295" y="0.375" size="1.27" layer="27" rot="R0.1"/>
 </element>
-<element name="C13" library="rcl" library_urn="urn:adsk.eagle:library:334" package="C0402" package3d_urn="urn:adsk.eagle:package:23626/1" value="0.1u" x="3.7" y="13.46" smashed="yes" rot="R90">
-<attribute name="NAME" x="3.765" y="15.725" size="1.27" layer="25" rot="R90"/>
-<attribute name="VALUE" x="6.305" y="12.025" size="1.27" layer="27" rot="R90"/>
+<element name="C13" library="rcl" library_urn="urn:adsk.eagle:library:334" package="C0402" package3d_urn="urn:adsk.eagle:package:23626/1" value="0.1u" x="1.9" y="12.96" smashed="yes" rot="R90">
+<attribute name="NAME" x="1.965" y="15.225" size="1.27" layer="25" rot="R90"/>
+<attribute name="VALUE" x="4.505" y="11.525" size="1.27" layer="27" rot="R90"/>
 </element>
 <element name="R4" library="rcl" library_urn="urn:adsk.eagle:library:334" package="M1206" package3d_urn="urn:adsk.eagle:package:23566/1" value="1.87k" x="30.5" y="4.06" smashed="yes" rot="R90">
@@
 <wire x1="23.6858" y1="42.2142" x2="23.5892625" y2="42.2142" width="0.508" layer="1"/>
 <wire x1="15.8074" y1="44.5" x2="21.3034625" y2="44.5" width="0.508" layer="1"/>
-<wire x1="23.5892625" y1="42.2142" x2="21.3034625" y2="44.5" width="0.508" layer="1"/>
+<wire x1="22.05173125" y1="43.75173125" x2="23.5892625" y2="42.2142" width="0.508" layer="1"/>
+<wire x1="22.05173125" y1="43.75173125" x2="21.3034625" y2="44.5" width="0.508" layer="1"/>
 <wire x1="19.7034625" y1="46.1" x2="21.3034625" y2="44.5" width="0.508" layer="1"/>
 <wire x1="19.7034625" y1="46.1" x2="15.8074" y2="46.1" width="0.508" layer="1"/>
@@
 <wire x1="16" y1="50.1" x2="16" y2="55.4" width="0.508" layer="1"/>
 <wire x1="16" y1="55.4" x2="18.8" y2="58.2" width="0.508" layer="1"/>
+<contactref element="U1" pad="18"/>
+<wire x1="24.3926" y1="43.7" x2="22.1034625" y2="43.7" width="0.508" layer="1"/>
+<wire x1="22.1034625" y1="43.7" x2="22.05173125" y2="43.75173125" width="0.508" layer="1"/>
 </signal>
 <signal name="GND">
@@
 <contactref element="C9" pad="2"/>
 <polygon width="0.1524" layer="1">
-<vertex x="-3.4" y="108.3"/>
-<vertex x="-15.4" y="96.3"/>
-<vertex x="-15.4" y="-14.5"/>
-<vertex x="-12.6" y="-11.7"/>
-<vertex x="174.1" y="-11.7"/>
-<vertex x="170.9" y="-8.5"/>
-<vertex x="170.9" y="116.4"/>
-<vertex x="162.8" y="108.3"/>
+<vertex x="8.6" y="99.9"/>
+<vertex x="0.1" y="100"/>
+<vertex x="0.2" y="0.1"/>
+<vertex x="2.6" y="0.2"/>
+<vertex x="102.5" y="0"/>
+<vertex x="102.5" y="4.6"/>
+<vertex x="102.3" y="99.9"/>
+<vertex x="87.1" y="99.8"/>
 </polygon>
 <polygon width="0.1524" layer="16">
-<vertex x="-5.2" y="104.9"/>
-<vertex x="-5.2" y="-6.7"/>
-<vertex x="-4.3" y="-5.8"/>
-<vertex x="166.9" y="-5.8"/>
-<vertex x="168.4" y="-4.3"/>
-<vertex x="168.4" y="103.4"/>
-<vertex x="-3.7" y="103.4"/>
+<vertex x="0.1" y="100"/>
+<vertex x="0.1" y="0.1"/>
+<vertex x="8.7" y="0.2"/>
+<vertex x="102.4" y="0"/>
+<vertex x="102.5" y="0.7"/>
+<vertex x="102.3" y="99.8"/>
+<vertex x="5.7" y="100"/>
 </polygon>
 <via x="18.7" y="47.3" extent="1-16" drill="0.35"/>
@@
 <via x="45" y="57.9" extent="1-16" drill="0.35"/>
 <via x="18" y="75.4" extent="1-16" drill="0.35"/>
-<via x="101.6" y="14.2" extent="1-16" drill="0.35"/>
+<via x="100" y="15.1" extent="1-16" drill="0.35"/>
 <via x="64.8" y="8.1" extent="1-16" drill="0.35"/>
 <via x="84.2" y="8.3" extent="1-16" drill="0.35"/>
@@
 <contactref element="R3" pad="1"/>
 <contactref element="BATTERY" pad="1"/>
-<polygon width="0.1524" layer="16">
-<vertex x="-3.2" y="100.3"/>
-<vertex x="-7.6" y="95.9"/>
-<vertex x="-7.6" y="-4.7"/>
-<vertex x="-6" y="-6.3"/>
-<vertex x="166.7" y="-6.3"/>
-<vertex x="173.1" y="0.1"/>
-<vertex x="173.1" y="103.4"/>
-<vertex x="-0.2" y="103.4"/>
-<vertex x="-3.3" y="100.3"/>
-</polygon>
 <contactref element="U1" pad="3"/>
 <contactref element="U1" pad="5"/>
@@
 <via x="23.9" y="50.8" extent="1-16" drill="0.35"/>
 <via x="24" y="41.1" extent="1-16" drill="0.35"/>
+<via x="81.7" y="38.5" extent="1-16" drill="0.35"/>
 </signal>
 <signal name="MISO">
@@
 <contactref element="D8" pad="A"/>
 <wire x1="8.7" y1="7.7" x2="11.04" y2="7.7" width="0.508" layer="1"/>
-<wire x1="8.7" y1="7.7" x2="6.385" y2="7.7" width="0.508" layer="1"/>
+<wire x1="8.7" y1="7.7" x2="4.685" y2="7.7" width="0.508" layer="1"/>
 <wire x1="11.04" y1="7.7" x2="11.04" y2="3" width="0.508" layer="1"/>
 <wire x1="26.5" y1="8.1" x2="24.7" y2="8.1" width="0.254" layer="1"/>
@@
 <contactref element="J2" pad="SHIELD1"/>
 <contactref element="C13" pad="1"/>
-<wire x1="3.7" y1="12.81" x2="3.7" y2="10.125" width="0.8128" layer="1"/>
-<wire x1="3.7" y1="10.125" x2="3.66" y2="10.085" width="0.8128" layer="1"/>
-<wire x1="3.66" y1="10.085" x2="3.66" y2="6.4" width="0.8128" layer="1"/>
-<wire x1="3.66" y1="6.4" x2="3.66" y2="2.715" width="0.8128" layer="1"/>
+<wire x1="1.9" y1="12.31" x2="1.9" y2="10.925" width="0.8128" layer="1"/>
+<wire x1="1.9" y1="10.925" x2="1.96" y2="10.085" width="0.8128" layer="1"/>
+<wire x1="1.96" y1="10.085" x2="1.96" y2="6.4" width="0.8128" layer="1"/>
+<wire x1="1.96" y1="6.4" x2="1.96" y2="2.715" width="0.8128" layer="1"/>
 </signal>
 <signal name="SCK">
