File: takpad6.2.brd (EAGLE design)
At the start: 102.6 x 100.1 mm, 75 parts, among them J1 SD_CARD_SOCKET, J10 AUDIO_JACK_TRRSSMD_RA, J3 AVR_SPI_PROG_3X2PTH, T1 0, T3 0, U1 ATMEGA328P_TQFP, U4 LM386N, Y1 20MHz

Commit message: Add files via upload
Parts:
- removed C22, C24: 1uF, SparkFun-Capacitors:0603
- added C17, C21: 1uF, SparkFun-Capacitors:0603
- added TP10, TP11, TP12, TP13, TP14, TP15, TP5, TP6, TP7, TP8, TP9: TPPAD1-17, testpad:P1-17
- added TP16, TP17: TPB1,27, testpad:B1,27
- TP1, TP4: value TPPAD1-17 -> TPB1,27; device testpad:P1-17 -> testpad:B1,27
- moved R14 142.6 mm to (38.0, 71.9), turned to 90 degrees
- moved R13 131.9 mm to (40.9, 66.4)
- moved R11 131.8 mm to (70.9, 64.2)
- moved R12 126.7 mm to (51.9, 62.8)
- moved R9 125.6 mm to (70.8, 70.0)
- moved R8 122.4 mm to (87.1, 57.6)
- moved R7 121.1 mm to (87.1, 62.2)
- moved R10 119.7 mm to (54.9, 66.6)
- moved TP4 107.9 mm to (-40.8, -106.4)
- moved TP1 78.7 mm to (-63.7, -116.7)
- moved C23 70.8 mm to (-13.1, -115.7)
Connections:
- removed net N$2: C23.2, U1.4
- removed net N$3: C22.2, U1.18
- removed net N$4: C24.2, U1.6
- net BAT: now also TP1.TP
- net GND: now also C17.1, C21.1, C23.1
- net PB6: now also TP13.TP
- net PB7: now also TP14.TP
- net RST: now also TP15.TP
- net SENS1LED: now also TP9.TP
- net SENS2LED: now also TP10.TP
- net SENS3LED: now also TP11.TP
- net SENS4LED: now also TP12.TP
- net SENSOR1OUT: now also TP8.TP
- net SENSOR2OUT: now also TP7.TP
- net SENSOR3OUT: now also TP6.TP
- net SENSOR4OUT: now also TP5.TP
- net TEMPSENSE: now also TP17.TP
- net V+: now also C17.2, C21.2, C23.2, U1.18, U1.4, U1.6; no longer C22.1, C23.1, C24.1, TP1.TP
- net VIN: now also TP16.TP
Routing:
- net V+: track 116.8 -> 125.3 mm
- net PD4: track 17.4 -> 18.4 mm

Commit message: Add files via upload
TO DO LIST:

MAJOR - 0.1uF caps by voltage pins - done (some of these are 1uF, is this the right value?)

Label pinouts, (not really sure what I am supposed to label)

change a few font sizes

some routing

some TP placement
Parts:
- TP10, TP11, TP12, TP13, TP14, TP15, TP2, TP3, TP5, TP6, TP7, TP8, TP9: value TPPAD1-17 -> TPB1,27; device testpad:P1-17 -> testpad:B1,27
- moved TP14 209.8 mm to (23.7, 29.9)
- moved TP12 206.8 mm to (9.40, 49.1)
- moved TP10 192.2 mm to (63.2, 39.6)
- moved C20 190.5 mm to (80.0, 4.90), turned to 180 degrees
- moved TP9 184.7 mm to (61.5, 43.6)
- moved TP11 182.6 mm to (56.7, 37.5)
- moved TP1 181.8 mm to (21.9, 43.7)
- moved TP13 181.8 mm to (13.2, 60.9)
- moved TP15 181.8 mm to (38.6, 6.00)
- moved TP6 175.5 mm to (67.2, 43.5)
- moved TP7 149.9 mm to (58.9, 40.4)
- moved TP3 146.5 mm to (55.0, 6.50)
- moved TP8 145.1 mm to (57.4, 43.9)
- moved TP4 134.8 mm to (17.0, 15.4)
- moved C23 134.2 mm to (11.9, 16.1)
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Routing:
- net SENSOR1OUT: track 71.6 -> 84.0 mm
- net N$1: track 4.00 -> 12.8 mm
- net V+: track 125.3 -> 122.6 mm
Other:
- board text added: "AAT3693"

Commit message: Add files via upload
Parts:
- added C22: 10uF, SparkFun-Capacitors:CPOL-RADIAL-2.5MM-5MM-KIT
- added C24: 0.1uF, SparkFun-Capacitors:CPOL-RADIAL-2.5MM-5MM-KIT
- moved TP11 56.4 mm to (51.1, 93.6)
- moved TP10 54.2 mm to (66.9, 93.7)
- moved TP9 53.7 mm to (80.9, 93.7)
- moved TP12 52.1 mm to (36.9, 93.3)
- moved TP15 37.8 mm to (40.4, 43.8)
- moved TP1 34.3 mm to (32.1, 10.9)
- moved C23 32.3 mm to (28.3, 43.9), turned to 180 degrees
- moved TP8 31.2 mm to (88.5, 45.7)
- moved TP7 21.9 mm to (67.5, 60.5)
- moved TP13 21.1 mm to (13.0, 39.8)
- moved TP6 21.1 mm to (53.6, 59.6)
- moved TP3 12.7 mm to (43.8, 12.4)
- moved TP5 12.3 mm to (43.0, 66.4)
- moved TP17 10.4 mm to (33.6, 9.50)
- moved T3 5.40 mm to (94.3, 69.1)
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Connections:
- new net BYPASS: C24.1, U4.7
- net GND: now also C22.2, C24.2
- net UPCONVERTERINPUT: now also C22.1
Routing:
- net V+: track 122.6 -> 141.3 mm
- net AUDIOOUT: track 3.45 -> 12.4 mm
- net UPCONVERTERINPUT: track 38.1 -> 45.7 mm
- net BYPASS: track 0.00 -> 7.07 mm
- net SCK: track 49.4 -> 55.7 mm
- net SENSOR4OUT: track 32.4 -> 37.5 mm
- net SENSOR1OUT: track 84.0 -> 87.8 mm
- net SENSOR2IN: track 7.74 -> 11.4 mm
- net SENSOR1IN: track 15.9 -> 19.4 mm
- net SENS2LED: track 77.9 -> 81.3 mm, vias 2 -> 4
- net SENSOR3IN: track 11.5 -> 14.7 mm
- net SENSOR3OUT: track 50.1 -> 46.8 mm
- net SENS1LED: track 84.3 -> 87.4 mm
- net RST: track 29.1 -> 32.1 mm
- net VIN: track 41.0 -> 43.9 mm
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
Commit message: Add files via upload
nearly done hope this works, cross fingers
Parts:
- added T2: 0, SparkFun-Resistors:AXIAL-0.3
Connections:
- net SENSOR1IN: now also T2.P$2
- net SENSOR1OUT: now also T2.P$1
Routing:
- net SENSOR1OUT: track 87.8 -> 94.7 mm
- net SENSOR1IN: track 19.4 -> 25.8 mm
